Commit message: Fully Working System

File: ros2_ws/src/gazebo_hello/urdf/camera.xacro (robot description, xacro)
@@ -30,38 +30,23 @@
     </joint>
     <gazebo reference="camera_link">
-        <sensor name="camera" type="camera">
-        <always_on>true</always_on>
+      <sensor name="camera" type="camera">
+        <pose>0 0 0 0 0 0</pose>
         <visualize>true</visualize>
         <update_rate>30</update_rate>
-        <camera name="intel_realsense_r200">
-          <horizontal_fov>1.02974</horizontal_fov>
+        <camera>
+          <horizontal_fov>1.0</horizontal_fov>
           <image>
-            <width>1920</width>
-            <height>1080</height>
+            <width>640</width>
+            <height>480</height>
             <format>R8G8B8</format>
           </image>
           <clip>
-            <near>0.02</near>
-            <far>300</far>
+            <near>0.05</near>
+            <far>100</far>
           </clip>
-          <noise>
-            <type>gaussian</type>
-            <!-- Noise is sampled independently per pixel on each frame.
-                  That pixel's noise value is added to each of its color
-                  channels, which at that point lie in the range [0,1]. -->
-            <mean>0.0</mean>
-            <stddev>0.007</stddev>
-          </noise>
         </camera>
-          <plugin name="camera_driver" filename="libgazebo_ros_camera.so">
-            <ros>
-              <!-- <namespace>test_cam</namespace> -->
-              <!-- <remapping>image_raw:=image_demo</remapping> -->
-              <!-- <remapping>camera_info:=camera_info_demo</remapping> -->
-            </ros>
-            <!-- camera_name>omit so it defaults to sensor name</camera_name-->
-            <!-- frame_name>omit so it defaults to link name</frameName-->
-            <!-- <hack_baseline>0.07</hack_baseline> -->
-          </plugin>
+        <plugin name="camera_driver" filename="libgazebo_ros_camera.so">
+          <frame_name>camera_link</frame_name>
+        </plugin>
       </sensor>
     </gazebo>

File: ros2_ws/src/gazebo_hello/urdf/example_gazebo.xacro (robot description, xacro)
@@ -26,6 +26,5 @@
     </gazebo>
     <!-- Plugin to receive JointTrajectory messages on /set_joint_trajectory
-         and move the robot accordingly (same as your example, but now for
-         pan_joint and tilt_joint). -->
+         and move the robot accordingly -->
     <gazebo>
         <plugin name="gazebo_ros_joint_pose_trajectory"
@@ -34,38 +33,3 @@
         </plugin>
     </gazebo>
-    <!-- Optional: depth camera on the camera_link, using a proper optical frame -->
-    <joint name="camera_optical_joint" type="fixed">
-        <origin xyz="0 0 0" rpy="-1.571 0 -1.571" />
-        <parent link="camera_link" />
-        <child link="camera_link_optical" />
-    </joint>
-    <link name="camera_link_optical"></link>
-    <gazebo reference="camera_link">
-        <sensor type="depth" name="my_camera">
-            <update_rate>20</update_rate>
-            <visualize>true</visualize>
-            <camera name="cam">
-                <horizontal_fov>1.3962634</horizontal_fov>
-                <image>
-                    <width>640</width>
-                    <height>480</height>
-                    <format>R8B8G8</format>
-                </image>
-                <clip>
-                    <near>0.02</near>
-                    <far>300</far>
-                </clip>
-                <noise>
-                    <type>gaussian</type>
-                    <mean>0.0</mean>
-                    <stddev>0.007</stddev>
-                </noise>
-            </camera>
-            <plugin name="camera_controller" filename="libgazebo_ros_camera.so">
-                <frame_name>camera_link_optical</frame_name>
-                <min_depth>0.1</min_depth>
-                <max_depth>500</max_depth>
-            </plugin>
-        </sensor>
-    </gazebo>
 </robot>
