Commit message: good commit

File: ros2_ws/src/gazebo_hello/urdf/example_include.xacro (robot description, xacro)
@@ -11,4 +11,7 @@
     <material name="blue">
         <color rgba="0.2 0.2 1 1"/>
+    </material>
+    <material name="black">
+        <color rgba="0.01 0.01 0.01 1"/>
     </material>
     <!-- Specify some standard inertial calculations https://en.wikipedia.org/wiki/List_of_moments_of_inertia -->

File: ros2_ws/src/gazebo_hello/urdf/pan_tilt.urdf.xacro (robot description, xacro)
@@ -8,5 +8,5 @@
     <!-- Fixed joint from world to base_link (like the example) -->
     <joint name="base_joint" type="fixed">
-        <origin xyz="0 0 0" rpy="0 0 0"/>
+        <origin xyz="0.081932 1.347850 0.5" rpy="0 0 0"/>
         <parent link="world"/>
         <child link="base_link"/>
