Commit message: moving face prismatic working for vertical

File: ros2_ws/src/gazebo_hello/urdf/moving_face.urdf (robot description, URDF)
Before this commit: robot moving_face, 3 links, 2 joints
Links:
- removed link base_link
- removed link left_wheel_link
- removed link right_wheel_link
- added link cube_link, mass 1.0; collision box size=0.2 0.2 0.2; visual box size=0.2 0.2 0.2
- added link lil_cube, mass 1.0; collision box size=0.01 0.01 0.01; visual box size=0.01 0.01 0.01
Joints:
- removed joint left_wheel_joint
- removed joint right_wheel_joint
- added joint prism_joint: type prismatic, parent lil_cube, child cube_link, origin xyz=0 0 0.05 rpy=0 0 0, axis 0 0 1, limit lower=-3.14159 upper=3.14159 effort=10 velocity=2.0

Commit message: Finished Project

File: ros2_ws/src/gazebo_hello/urdf/moving_face.urdf (robot description, URDF)
Before this commit: robot moving_face, 2 links, 1 joints
Links:
- removed link lil_cube
- added link x_cube, mass 1.0; collision box size=0.01 0.01 0.01; visual box size=0.01 0.01 0.01
- added link z_cube, mass 1.0; collision box size=0.01 0.01 0.01; visual box size=0.01 0.01 0.01
Joints:
- removed joint prism_joint
- added joint x_joint: type prismatic, parent x_cube, child cube_link, origin xyz=0 0 0.05 rpy=0 0 0, axis 1 0 0, limit lower=-0.5 upper=0.5 effort=10 velocity=2.0
- added joint z_joint: type prismatic, parent z_cube, child x_cube, origin xyz=0 0 0.05 rpy=0 0 0, axis 0 0 1, limit lower=-0.5 upper=0.5 effort=10 velocity=2.0
